Commit message: fix: stompy trained on all AMASS data.

File: legged_gym/resources/robots/stompypro/robot_test.urdf (robot description, URDF)
Before this commit: robot robot, 19 links, 18 joints
Joints:
- joint L_ankle_y: limit lower=-0.698 upper=0.698 effort=17 velocity=20 -> lower=-3.14 upper=3.14 effort=17 velocity=20
- joint L_elbow_x: limit lower=-1.9199 upper=1.9199 effort=17 velocity=20 -> lower=-3.14 upper=3.14 effort=17 velocity=20
- joint L_hip_x: limit lower=-0.523 upper=2.093 effort=120 velocity=20 -> lower=-3.14 upper=3.14 effort=120 velocity=20
- joint L_knee: limit lower=-1.919 upper=1.919 effort=200 velocity=20 -> lower=-3.14 upper=3.14 effort=200 velocity=20
- joint L_shoulder_x: limit lower=0 upper=3.1416 effort=60 velocity=20 -> lower=-3.14 upper=3.1416 effort=60 velocity=20
- joint L_shoulder_y: limit lower=-3.1416 upper=3.1416 effort=60 velocity=20 -> lower=-3.14 upper=3.1416 effort=60 velocity=20
- joint R_ankle_y: limit lower=-0.698 upper=0.698 effort=17 velocity=20 -> lower=-3.14 upper=3.14 effort=17 velocity=20
- joint R_elbow_x: limit lower=-1.9199 upper=1.9199 effort=17 velocity=20 -> lower=-3.14 upper=3.14 effort=17 velocity=20
- joint R_hip_x: limit lower=-2.093 upper=0.523 effort=120 velocity=20 -> lower=-3.14 upper=3.14 effort=120 velocity=20
- joint R_knee: limit lower=-1.919 upper=1.919 effort=200 velocity=20 -> lower=-3.14 upper=3.14 effort=200 velocity=20
- joint R_shoulder_x: limit lower=-3.1416 upper=0 effort=60 velocity=20 -> lower=-3.14 upper=3.14 effort=60 velocity=20
- joint R_shoulder_y: limit lower=-3.1416 upper=3.1416 effort=60 velocity=20 -> lower=-3.14 upper=3.1416 effort=60 velocity=20
